Commit message: Updated novamx

File: robot.urdf (robot description, URDF)
Before this commit: robot mini_sumo, 5 links, 4 joints
Joints:
- joint nose_wedge_joint: origin xyz=0.0500 0.0 0.0052 rpy=0 0.3672 0 -> xyz=0.0500 0.0 0.0058 rpy=0 0.3672 0

Commit message: Updated agent's model

File: robot.urdf (robot description, URDF)
Before this commit: robot mini_sumo, 5 links, 4 joints
Links:
- link base_link: mass 0.4 -> 0.45; geometry collision box size=0.0822 0.098 0.040; visual box size=0.0822 0.098 0.040
- link left_wheel: mass 0.05 -> 0.025; geometry collision cylinder length=0.019 radius=0.010; visual cylinder length=0.019 radius=0.010
- link nose_wedge: geometry collision box size=0.01948 0.098 0.002; visual box size=0.01948 0.098 0.002
- link right_wheel: mass 0.05 -> 0.025; geometry collision cylinder length=0.019 radius=0.010; visual cylinder length=0.019 radius=0.010
Joints:
- joint front_caster_joint: origin xyz=0.045 0.0 0.003 rpy=0 0 0 -> xyz=0.025 0.0 0.003 rpy=0 0 0
- joint left_wheel_joint: origin xyz=-0.0387 0.028 0.014 rpy=0 0 0 -> xyz=-0.025 0.0401 0.010 rpy=0 0 0
- joint nose_wedge_joint: origin xyz=0.0500 0.0 0.0058 rpy=0 0.3672 0 -> xyz=0.0411 0.0 0.0061 rpy=0 0.5101 0
- joint right_wheel_joint: origin xyz=-0.0387 -0.028 0.014 rpy=0 0 0 -> xyz=-0.025 -0.0401 0.010 rpy=0 0 0
